Commit message: finish changes in description URDFs, insert gripperCam moveit

File: open_manipulator_p_description/urdf/bir_open_manipulator_p.urdf.xacro (robot description, xacro)
@@ -123,5 +123,5 @@
     <parent link="link3"/>
     <child link="link4"/>
-    <origin xyz="0.03000 0.0 0.26400" rpy="0 0 0"/>
+    <origin xyz="0.03000 0.0 0.26400" rpy="0 -0.7854 0"/>
     <axis xyz="0 1 0"/>
     <limit velocity="0.31415" effort="1000" lower="${-pi*60/180}" upper="${pi*120/180}" />

File: open_manipulator_p_description/urdf/bir_open_manipulator_p_with_cam.urdf.xacro (robot description, xacro)
@@ -163,5 +163,5 @@
     <parent link="link3"/>
     <child link="link4"/>
-    <origin xyz="0.03000 0.0 0.26400" rpy="0 0 0"/>
+    <origin xyz="0.03000 0.0 0.26400" rpy="0 -0.7854 0"/>
     <axis xyz="0 1 0"/>
     <limit velocity="0.31415" effort="1000" lower="${-pi*60/180}" upper="${pi*120/180}" />
@@ -305,5 +305,5 @@
       <origin xyz="0 0 1.557" rpy="0 0 0"/>
       <geometry>
-        <mesh filename="package://open_manipulator_pro_description/meshes/bir_camera_with_base_lens.dae"/>
+        <mesh filename="package://open_manipulator_p_description/meshes/bir_camera_with_base_lens.dae"/>
       </geometry>
     </collision>
@@ -311,5 +311,5 @@
       <origin rpy="0 0 1.557" xyz="0 0 0"/>
       <geometry>
-        <mesh filename="package://open_manipulator_pro_description/meshes/bir_camera_with_base_lens.dae"/>
+        <mesh filename="package://open_manipulator_p_description/meshes/bir_camera_with_base_lens.dae"/>
       </geometry>
     </visual>

File: open_manipulator_p_description/urdf/bir_open_manipulator_p_with_gripper_cam.urdf.xacro (robot description, xacro)
@@ -163,5 +163,5 @@
     <parent link="link3"/>
     <child link="link4"/>
-    <origin xyz="0.03000 0.0 0.26400" rpy="0 0 0"/>
+    <origin xyz="0.03000 0.0 0.26400" rpy="0 -0.7854 0"/>
     <axis xyz="0 1 0"/>
     <limit velocity="0.31415" effort="1000" lower="${-pi*60/180}" upper="${pi*120/180}" />
@@ -276,5 +276,5 @@
       <origin rpy="0 0 3.1415" xyz="0.073 0.014 -0.024"/>
       <geometry>
-        <mesh filename="package://open_manipulator_pro_description/meshes/bir_gripperMX_fixed.dae"/>
+        <mesh filename="package://open_manipulator_p_description/meshes/bir_gripperMX_fixed.dae"/>
       </geometry>
     </collision>
@@ -282,5 +282,5 @@
       <origin rpy="0 0 3.1415" xyz="0.073 0.014 -0.024"/>
       <geometry>
-        <mesh filename="package://open_manipulator_pro_description/meshes/bir_gripperMX_fixed.dae"/>
+        <mesh filename="package://open_manipulator_p_description/meshes/bir_gripperMX_fixed.dae"/>
       </geometry>
     </visual>
@@ -309,5 +309,5 @@
     <origin rpy="0 0 3.1415" xyz="0 0 0"/>
     <geometry>
-      <mesh filename="package://open_manipulator_pro_description/meshes/bir_gripperMX_claw.dae"/>
+      <mesh filename="package://open_manipulator_p_description/meshes/bir_gripperMX_claw.dae"/>
     </geometry>
   </collision>
@@ -315,5 +315,5 @@
     <origin rpy="0 0 3.1415" xyz="0 0 0"/>
     <geometry>
-      <mesh filename="package://open_manipulator_pro_description/meshes/bir_gripperMX_claw.dae"/>
+      <mesh filename="package://open_manipulator_p_description/meshes/bir_gripperMX_claw.dae"/>
     </geometry>
     <material name="grey"/>
@@ -330,5 +330,5 @@
       <origin xyz="0 0 1.557" rpy="0 0 0"/>
       <geometry>
-        <mesh filename="package://open_manipulator_pro_description/meshes/bir_camera_with_base_lens.dae"/>
+        <mesh filename="package://open_manipulator_p_description/meshes/bir_camera_with_base_lens.dae"/>
       </geometry>
     </collision>
@@ -336,5 +336,5 @@
       <origin rpy="0 0 1.557" xyz="0 0 0"/>
       <geometry>
-        <mesh filename="package://open_manipulator_pro_description/meshes/bir_camera_with_base_lens.dae"/>
+        <mesh filename="package://open_manipulator_p_description/meshes/bir_camera_with_base_lens.dae"/>
       </geometry>
     </visual>

Commit message: insert changes in J3 to match real position

File: open_manipulator_p_description/urdf/bir_open_manipulator_p.urdf.xacro (robot description, xacro)
@@ -124,4 +124,5 @@
     <child link="link4"/>
     <origin xyz="0.03000 0.0 0.26400" rpy="0 -0.7854 0"/>
+    <!--<origin xyz="0.03000 0.0 0.26400" rpy="0 0 0"/>-->
     <axis xyz="0 1 0"/>
     <limit velocity="0.31415" effort="1000" lower="${-pi*60/180}" upper="${pi*120/180}" />

File: open_manipulator_p_description/urdf/bir_open_manipulator_p_with_cam.urdf.xacro (robot description, xacro)
@@ -164,4 +164,5 @@
     <child link="link4"/>
     <origin xyz="0.03000 0.0 0.26400" rpy="0 -0.7854 0"/>
+    <!--<origin xyz="0.03000 0.0 0.26400" rpy="0 0 0"/>-->
     <axis xyz="0 1 0"/>
     <limit velocity="0.31415" effort="1000" lower="${-pi*60/180}" upper="${pi*120/180}" />

File: open_manipulator_p_description/urdf/bir_open_manipulator_p_with_gripper_cam.urdf.xacro (robot description, xacro)
@@ -164,4 +164,5 @@
     <child link="link4"/>
     <origin xyz="0.03000 0.0 0.26400" rpy="0 -0.7854 0"/>
+    <!--<origin xyz="0.03000 0.0 0.26400" rpy="0 0 0"/>-->
     <axis xyz="0 1 0"/>
     <limit velocity="0.31415" effort="1000" lower="${-pi*60/180}" upper="${pi*120/180}" />

Commit message: insert J1 limits +-90 to avoid broken cables

File: open_manipulator_p_description/urdf/bir_open_manipulator_p.urdf.xacro (robot description, xacro)
@@ -58,5 +58,5 @@
     <origin xyz="0.0 0.0 0.126" rpy="0 0 0"/>
     <axis xyz="0 0 1"/>
-    <limit velocity="0.31415" effort="1000" lower="${-pi*175/180}" upper="${pi*175/180}"/>
+    <limit velocity="0.31415" effort="1000" lower="${-pi*90/180}" upper="${pi*90/180}"/>
     <dynamics damping="0.7"/>
   </joint>

File: open_manipulator_p_description/urdf/bir_open_manipulator_p_with_cam.urdf.xacro (robot description, xacro)
@@ -98,5 +98,5 @@
     <origin xyz="0.0 0.0 0.126" rpy="0 0 0"/>
     <axis xyz="0 0 1"/>
-    <limit velocity="0.31415" effort="1000" lower="${-pi*175/180}" upper="${pi*175/180}"/>
+    <limit velocity="0.31415" effort="1000" lower="${-pi*90/180}" upper="${pi*90/180}"/>
     <dynamics damping="0.7"/>
   </joint>

File: open_manipulator_p_description/urdf/bir_open_manipulator_p_with_gripper_cam.urdf.xacro (robot description, xacro)
@@ -98,5 +98,5 @@
     <origin xyz="0.0 0.0 0.126" rpy="0 0 0"/>
     <axis xyz="0 0 1"/>
-    <limit velocity="0.31415" effort="1000" lower="${-pi*175/180}" upper="${pi*175/180}"/>
+    <limit velocity="0.31415" effort="1000" lower="${-pi*90/180}" upper="${pi*90/180}"/>
     <dynamics damping="0.7"/>
   </joint>
